File: Rev.0/kicad/breakout.kicad_pcb (KiCad board)
At the start: 2 copper layers, 63.5 x 77.2 mm, 40 parts, among them J1 Conn_02x10_Odd_Even, J10 Conn_02x10_Odd_Even, J12 Conn_02x10_Odd_Even, J2 Conn_02x10_Odd_Even, J3 Conn_01x02, J4 Conn_01x03_Pin, J5 Conn_01x05_Pin, M1 MountingHole_3.5mm_Pad_TopBot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, M2 MountingHole_3.5mm_Pad_TopBot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, U1 RP2040Z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

Commit message: Rev.0: corrected U1 to WaveShare RP2040-TINY
Parts:
- U1: value RP2040Z -> RP2040-TINY; footprint uhppoted:RP2040Z -> uhppoted:RP2040-TINY
Changed lines of the file:
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@@
     )
   )
-  (footprint "uhppoted:RP2040Z" (layer "F.Cu")
+  (footprint "uhppoted:RP2040-TINY" (layer "F.Cu")
     (at 106.75 136.46)
     (property "Sheetfile" "breakout.kicad_sch")
@@
         (effects (font (size 1 1) (thickness 0.15)))
     )
-    (fp_text value "RP2040Z" (at 0 0 unlocked) (layer "F.Fab")
+    (fp_text value "RP2040-TINY" (at 0 0 unlocked) (layer "F.Fab") hide
         (effects (font (size 1 1) (thickness 0.15)))
     )
-    (fp_text user "${REFERENCE}" (at 0 2 unlocked) (layer "F.Fab")
+    (fp_text user "${REFERENCE}" (at 0 2 unlocked) (layer "F.Fab") hide
         (effects (font (size 1 1) (thickness 0.15)))
     )
@@
     (pad "23" thru_hole roundrect (at 7.62 -10.16) (size 2.6 1.6) (drill 0.8 (offset 0.6 0)) (layers "*.Cu" "*.Mask") (roundrect_rratio 0.25)
       (net 24 "/TX") (pinfunction "UART0 TX") (pintype "output"))
-    (model "${KICAD_UHPPOTED}/library/uhppoted.pretty/RP2040Z.step"
+    (model "${KICAD_UHPPOTED}/uhppoted.pretty/RP2040-TINY.step"
       (offset (xyz -8.95 -12.6 0))
       (scale (xyz 1 1 1))
