File: Rev.0/kicad/v0.1/breakout.kicad_pcb (KiCad board)
At the start: 2 copper layers, 63.5 x 77.2 mm, 40 parts, among them J1 Conn_02x10_Odd_Even, J10 Conn_02x10_Odd_Even, J12 Conn_02x10_Odd_Even, J2 Conn_02x10_Odd_Even, J3 Conn_01x02, J4 Conn_01x03_Pin, J5 Conn_01x05_Pin, M1 MountingHole_3.5mm_Pad_TopBot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, M2 MountingHole_3.5mm_Pad_TopBot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, U1 RP2040-TINY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

Commit message: Added RX8900SA battery diodes and resistors to flip side of PCB
Parts:
- added H1: MountingHole_2.1mm, MountingHole:MountingHole_2.1mm, F.Cu at (101.0, 118.8)
- added H2: MountingHole_2.1mm, MountingHole:MountingHole_2.1mm, F.Cu at (112.5, 118.8)
- added H3: MountingHole_2.1mm, MountingHole:MountingHole_2.1mm, F.Cu at (101.0, 165.8)
- added H4: MountingHole_2.1mm, MountingHole:MountingHole_2.1mm, F.Cu at (112.5, 165.8)
- D1, D2: footprint Diode_THT:D_DO-35_SOD27_P7.62mm_Horizontal -> Diode_SMD:D_SOD-123; moved to B.Cu
- R8: footprint Resistor_THT:R_Axial_DIN0207_L6.3mm_D2.5mm_P7.62mm_Horizontal -> Resistor_SMD:R_1206_3216Metric_Pad1.30x1.75mm_HandSolder; moved to B.Cu
- moved D2 8.03 mm to (96.6, 116.1), turned to -90 degrees
- moved D1 6.35 mm to (92.8, 116.1)
- moved R8 6.35 mm to (89.0, 116.1)
- moved G*** 5.68 mm to (118.2, 166.9)
- moved C1 1.80 mm to (100.4, 112.3)
- moved C8 1.80 mm to (100.4, 107.2)
- moved U5 0.82 mm to (107.6, 108.5)
Routing:
- net Net-(D1-K): track 8.41 -> 16.0 mm, vias 0 -> 1
- net GND: track 34.2 -> 28.0 mm
- net Net-(BAT1-+): track 28.0 -> 33.1 mm, vias 0 -> 1
- net +3V3: track 126.7 -> 127.6 mm, vias 4 -> 3
- net Net-(D2-K): track 11.2 -> 10.3 mm, vias 0 -> 1
- net /SDA1: track 88.0 -> 87.2 mm
- net /SCL1: track 95.5 -> 96.3 mm
Other:
- board text added: "BREAKOUT Rev.0.1"
- board text removed: "BREAKOUT Rev 0.1"
